Commit message: Update collision box and joint type.

File: urdf/b29/b29.urdf.xacro (robot description, xacro)
@@ -2,4 +2,8 @@
 <robot xmlns:xacro="http://www.ros.org/wiki/xacro" name="b29">
     <xacro:arg name="use_simulation" default="true"/>
+    <xacro:property name="wheel_radius" value="0.0405"/>
+    <xacro:property name="wheel_edge_radius" value="0.0460"/>
+    <xacro:property name="wheel_height" value="0.0153"/>
+    <xacro:property name="wheel_edge_height" value="0.002"/>
     <link name="base_link">
         <inertial>
@@ -15,7 +19,7 @@
         </visual>
         <collision>
-            <origin xyz="0 0 0" rpy="0 0 0"/>
-            <geometry>
-                <mesh filename="package://b29_control/meshes/b29/base_link.stl"/>
+            <origin xyz="0 -0.01 -0.017" rpy="0 0 0"/>
+            <geometry>
+                <box size="0.344 0.064 0.075"/>
             </geometry>
         </collision>
@@ -33,10 +37,4 @@
             </geometry>
         </visual>
-        <collision>
-            <origin xyz="0 0 0" rpy="0 0 0"/>
-            <geometry>
-                <mesh filename="package://b29_control/meshes/b29/left_first_leg.stl"/>
-            </geometry>
-        </collision>
     </link>
     <joint name="left_first_leg_joint" type="revolute">
@@ -146,7 +144,19 @@
         </visual>
         <collision>
-            <origin xyz="0 0.0 0.0" rpy="0 0 0"/>
-            <geometry>
-                <mesh filename="package://b29_control/meshes/b29/friction_wheel.stl"/>
+            <origin xyz="0 ${wheel_edge_height/2} 0" rpy="${-pi/2} 0 0"/>
+            <geometry>
+                <cylinder radius="${wheel_edge_radius}" length="${wheel_edge_height}"/>
+            </geometry>
+        </collision>
+        <collision>
+            <origin xyz="0 ${wheel_edge_height+wheel_height/2} 0" rpy="${-pi/2} 0 0"/>
+            <geometry>
+                <cylinder radius="${wheel_radius}" length="${wheel_height}"/>
+            </geometry>
+        </collision>
+        <collision>
+            <origin xyz="0 ${wheel_edge_height+wheel_height+wheel_edge_height/2} 0" rpy="${-pi/2} 0 0"/>
+            <geometry>
+                <cylinder radius="${wheel_edge_radius}" length="${wheel_edge_height}"/>
             </geometry>
         </collision>
@@ -173,10 +183,4 @@
             </geometry>
         </visual>
-        <collision>
-            <origin xyz="0 0 0" rpy="0 0 0"/>
-            <geometry>
-                <mesh filename="package://b29_control/meshes/b29/right_first_leg.stl"/>
-            </geometry>
-        </collision>
     </link>
     <joint name="right_first_leg_joint" type="revolute">
@@ -286,7 +290,19 @@
         </visual>
         <collision>
-            <origin xyz="0 0.0 0.0" rpy="0 0 0"/>
-            <geometry>
-                <mesh filename="package://b29_control/meshes/b29/friction_wheel.stl"/>
+            <origin xyz="0 ${wheel_edge_height/2} 0" rpy="${-pi/2} 0 0"/>
+            <geometry>
+                <cylinder radius="${wheel_edge_radius}" length="${wheel_edge_height}"/>
+            </geometry>
+        </collision>
+        <collision>
+            <origin xyz="0 ${wheel_edge_height+wheel_height/2} 0" rpy="${-pi/2} 0 0"/>
+            <geometry>
+                <cylinder radius="${wheel_radius}" length="${wheel_height}"/>
+            </geometry>
+        </collision>
+        <collision>
+            <origin xyz="0 ${wheel_edge_height+wheel_height+wheel_edge_height/2} 0" rpy="${-pi/2} 0 0"/>
+            <geometry>
+                <cylinder radius="${wheel_edge_radius}" length="${wheel_edge_height}"/>
             </geometry>
         </collision>
@@ -338,5 +354,5 @@
         <joint name="left_friction_wheel_joint">
             <offset>0</offset>
-            <hardwareInterface>hardware_interface/PositionJointInterface</hardwareInterface>
+            <hardwareInterface>hardware_interface/VelocityJointInterface</hardwareInterface>
         </joint>
     </transmission>
@@ -378,5 +394,5 @@
         <joint name="right_friction_wheel_joint">
             <offset>0</offset>
-            <hardwareInterface>hardware_interface/PositionJointInterface</hardwareInterface>
+            <hardwareInterface>hardware_interface/VelocityJointInterface</hardwareInterface>
         </joint>
     </transmission>

Commit message: Update conflict box and fix left_first_leg.

File: urdf/b29/b29.urdf.xacro (robot description, xacro)
@@ -21,5 +21,5 @@
             <origin xyz="0 -0.01 -0.017" rpy="0 0 0"/>
             <geometry>
-                <box size="0.344 0.064 0.075"/>
+                <box size="0.244 0.064 0.075"/>
             </geometry>
         </collision>
@@ -60,7 +60,7 @@
         </visual>
         <collision>
-            <origin xyz="0 0.0 0.0" rpy="0 0 0"/>
-            <geometry>
-                <mesh filename="package://b29_control/meshes/b29/second_leg.stl"/>
+            <origin xyz="0 -0.03 0.184" rpy="0 0 0"/>
+            <geometry>
+                <box size="0.1 0.002 0.26"/>
             </geometry>
         </collision>
@@ -206,7 +206,7 @@
         </visual>
         <collision>
-            <origin xyz="0 0.0 0.0" rpy="0 0 0"/>
-            <geometry>
-                <mesh filename="package://b29_control/meshes/b29/second_leg.stl"/>
+            <origin xyz="0 -0.03 0.184" rpy="0 0 0"/>
+            <geometry>
+                <box size="0.1 0.002 0.26"/>
             </geometry>
         </collision>
@@ -397,4 +397,11 @@
         </joint>
     </transmission>
+    <gazebo>
+        <joint name="world_fixed_joint" type="fixed">
+            <parent>world</parent>
+            <child>left_second_leg</child>
+            <pose>0 0 -0.25 0 0 0</pose>
+        </joint>
+    </gazebo>
     <xacro:if value="$(arg use_simulation)">
         <gazebo>
