Commit message: Update URDF.

File: b29_control/urdf/b29/b29.urdf.xacro (robot description, xacro)
@@ -6,4 +6,5 @@
     <xacro:property name="wheel_height" value="0.0153"/>
     <xacro:property name="wheel_edge_height" value="0.002"/>
+    <xacro:include filename="$(find b29_control)/urdf/common/imu.urdf.xacro"/>
     <link name="base_link">
         <inertial>
@@ -25,4 +26,6 @@
         </collision>
     </link>
+    <xacro:IMU connected_to="base_link" imu_name="base_imu" xyz="0.0 0.0 0.01"
+               rpy="0 0 0"/>
     <link name="left_first_leg">
         <inertial>
@@ -42,5 +45,5 @@
                 rpy="0 0 0"/>
         <dynamics damping="0.0" friction="0.1"/>
-        <limit effort="97" velocity="6.28" lower="-1e10" upper="1e10"/>
+        <limit effort="97" velocity="6.28" lower="${-pi}" upper="${pi}"/>
         <parent link="base_link"/>
         <child link="left_first_leg"/>
@@ -70,5 +73,5 @@
                 rpy="0 0 0"/>
         <dynamics damping="0.0" friction="0.1"/>
-        <limit effort="27" velocity="5.44" lower="-1e10" upper="1e10"/>
+        <limit effort="27" velocity="5.44" lower="${-pi}" upper="${pi}"/>
         <parent link="left_first_leg"/>
         <child link="left_second_leg"/>
@@ -188,5 +191,5 @@
                 rpy="0 0 0"/>
         <dynamics damping="0.0" friction="0.1"/>
-        <limit effort="97" velocity="6.28" lower="-1e10" upper="1e10"/>
+        <limit effort="97" velocity="6.28" lower="${-pi}" upper="${pi}"/>
         <parent link="base_link"/>
         <child link="right_first_leg"/>
@@ -216,5 +219,5 @@
                 rpy="0 0 0"/>
         <dynamics damping="0.0" friction="0.1"/>
-        <limit effort="27" velocity="5.44" lower="-1e10" upper="1e10"/>
+        <limit effort="27" velocity="5.44" lower="${-pi}" upper="${pi}"/>
         <parent link="right_first_leg"/>
         <child link="right_second_leg"/>

File: b29_control/urdf/common/imu.urdf.xacro (robot description, xacro)
@@ -18,5 +18,5 @@
                 <origin rpy="0 0 0" xyz="0 0 0"/>
                 <geometry>
-                    <mesh filename="package://rm_description/meshes/common/imu.stl" scale="1 1 1"/>
+                    <box size="0.03 0.02 0.005"/>
                 </geometry>
             </visual>

Commit message: Update URDF.

File: b29_control/urdf/b29/b29.urdf.xacro (robot description, xacro)
@@ -165,9 +165,9 @@
         </collision>
     </link>
-    <joint name="left_friction_wheel_joint" type="revolute">
+    <joint name="left_friction_wheel_joint" type="continuous">
         <origin xyz="0 0.012 0.2665"
                 rpy="0 0 0"/>
         <dynamics damping="0.0" friction="0.1"/>
-        <limit effort="3.42" velocity="73" lower="-1e10" upper="1e10"/>
+        <limit effort="3.42" velocity="73"/>
         <parent link="left_second_leg"/>
         <child link="left_friction_wheel"/>
@@ -311,9 +311,9 @@
         </collision>
     </link>
-    <joint name="right_friction_wheel_joint" type="revolute">
+    <joint name="right_friction_wheel_joint" type="continuous">
         <origin xyz="0 0.012 0.2665"
                 rpy="0 0 0"/>
         <dynamics damping="0.0" friction="0.1"/>
-        <limit effort="3.42" velocity="73" lower="-1e10" upper="1e10"/>
+        <limit effort="3.42" velocity="73"/>
         <parent link="right_second_leg"/>
         <child link="right_friction_wheel"/>

Commit message: Limit velocity.

File: b29_control/urdf/b29/b29.urdf.xacro (robot description, xacro)
@@ -41,5 +41,5 @@
         </visual>
     </link>
-    <joint name="left_first_leg_joint" type="revolute">
+    <joint name="left_first_leg_joint" type="continuous">
         <origin xyz="0.1689 -0.01425 -0.016"
                 rpy="0 0 0"/>
@@ -69,9 +69,9 @@
         </collision>
     </link>
-    <joint name="left_second_leg_joint" type="revolute">
+    <joint name="left_second_leg_joint" type="continuous">
         <origin xyz="0.050346 -0.03 0.04783"
                 rpy="0 0 0"/>
         <dynamics damping="0.0" friction="0.1"/>
-        <limit effort="27" velocity="5.44" lower="${-pi}" upper="${pi}"/>
+        <limit effort="27" velocity="1.44" lower="${-pi}" upper="${pi}"/>
         <parent link="left_first_leg"/>
         <child link="left_second_leg"/>
@@ -187,5 +187,5 @@
         </visual>
     </link>
-    <joint name="right_first_leg_joint" type="revolute">
+    <joint name="right_first_leg_joint" type="continuous">
         <origin xyz="-0.1312 -0.01425 -0.016"
                 rpy="0 0 0"/>
@@ -215,9 +215,9 @@
         </collision>
     </link>
-    <joint name="right_second_leg_joint" type="revolute">
+    <joint name="right_second_leg_joint" type="continuous">
         <origin xyz="-0.050346 -0.03 0.04783"
                 rpy="0 0 0"/>
         <dynamics damping="0.0" friction="0.1"/>
-        <limit effort="27" velocity="5.44" lower="${-pi}" upper="${pi}"/>
+        <limit effort="27" velocity="1.44" lower="${-pi}" upper="${pi}"/>
         <parent link="right_first_leg"/>
         <child link="right_second_leg"/>
