Commit message: 临时测试

File: b29_control/urdf/b29/b29.urdf.xacro (robot description, xacro)
@@ -45,5 +45,5 @@
     </link>
     <joint name="left_first_leg_joint" type="continuous">
-        <origin xyz="-0.299916107911189 -0.00183492089258142 0.0379999999994639" rpy="0 0 0"/>
+        <origin xyz="0.30008 0.0018349 0.038" rpy="0 0 0"/>
         <parent link="base_link"/>
         <child link="left_first_leg"/>
@@ -72,5 +72,5 @@
     </link>
     <joint name="left_second_leg_joint" type="continuous">
-        <origin xyz="-0.07 -0.01359 0.22765" rpy="0 0 0"/>
+        <origin xyz="0.07 -0.01359 0.22765" rpy="0 0 0"/>
         <parent link="left_first_leg"/>
         <child link="left_second_leg"/>
@@ -203,4 +203,5 @@
         <child link="l_gripper_right_up"/>
         <axis xyz="-1 0 0"/>
+        <mimic joint="l_gripper_left_drive_joint" multiplier="1" offset="0"/>
         <limit lower="-0.015" upper="0.015" effort="50" velocity="0.2"/>
         <dynamics damping="150.0" friction="5.0"/>
@@ -233,5 +234,5 @@
     </link>
     <joint name="right_first_leg_joint" type="continuous">
-        <origin xyz="0.30008 0.0018349 0.038" rpy="0 0 0"/>
+        <origin xyz="-0.299916107911189 -0.00183492089258142 0.0379999999994639" rpy="0 0 0"/>
         <parent link="base_link"/>
         <child link="right_first_leg"/>
@@ -260,5 +261,5 @@
     </link>
     <joint name="right_second_leg_joint" type="continuous">
-        <origin xyz="0.07 -0.0018099 0.22765" rpy="0 0 0"/>
+        <origin xyz="-0.07 -0.0018099 0.22765" rpy="0 0 0"/>
         <parent link="right_first_leg"/>
         <child link="right_second_leg"/>
@@ -392,4 +393,5 @@
         <child link="r_gripper_right_uprod"/>
         <axis xyz="-1 0 0"/>
+        <mimic joint="r_gripper_left_drive_joint" multiplier="1" offset="0"/>
         <limit lower="-0.015" upper="0.015" effort="50" velocity="0.2"/>
         <dynamics damping="150.0" friction="5.0"/>
@@ -415,5 +417,5 @@
         <type>transmission_interface/SimpleTransmission</type>
         <actuator name="left_second_leg_motor">
-            <mechanicalReduction>1</mechanicalReduction>
+            <mechanicalReduction>-1</mechanicalReduction>
         </actuator>
         <joint name="left_second_leg_joint">
@@ -455,5 +457,5 @@
         <type>transmission_interface/SimpleTransmission</type>
         <actuator name="right_second_leg_motor">
-            <mechanicalReduction>1</mechanicalReduction>
+            <mechanicalReduction>-1</mechanicalReduction>
         </actuator>
         <joint name="right_second_leg_joint">
@@ -488,5 +490,5 @@
             <pose>0 0 -0.25 0 0 0</pose>
         </joint>
-    </gazebo>
+        </gazebo>
     <xacro:if value="$(arg use_simulation)">
         <gazebo>
